File: hardware/barometer-v2.kicad_pcb (KiCad board)
At the start: 2 copper layers, 15 x 25 mm, 26 parts, among them P1 CON-SENSOR2, P2 CONN_01X01, P3 BOOT, U1 XMC1XXX24, U2 LPS22HB, U3 DRILL, U4 DRILL, U5 DRILL, U6 DRILL

Commit message: fix logo positions
Parts:
- moved VAL 7.21 mm to (147.8, 109.1)
- moved G*** 3.75 mm to (147.8, 103.1)
- moved VAL 2.69 mm to (147.8, 97.6)
Changed lines of the file:
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@@
-(kicad_pcb (version 4) (host pcbnew 4.0.7-e2-6376~58~ubuntu17.04.1)
+(kicad_pcb (version 4) (host pcbnew 4.0.7-e2-6376~61~ubuntu18.04.1)
   (general
     (links 53)
@@
   (layers
     (0 Vorderseite signal)
-    (31 Rückseite signal hide)
+    (31 Rückseite signal)
     (32 B.Adhes user)
     (33 F.Adhes user)
@@
   )
   (setup
-    (last_trace_width 0.2)
+    (last_trace_width 0.29972)
     (user_trace_width 0.2)
     (user_trace_width 0.25)
@@
     (pad_drill 0)
     (pad_to_mask_clearance 0)
-    (aux_axis_origin 140.32484 115.62588)
+    (aux_axis_origin 140.3 90.6)
+    (grid_origin 140.3 90.6)
     (visible_elements FFFFFFBF)
     (pcbplotparams
@@
   )
   (module kicad-libraries:CE_5mm (layer Rückseite)
-    (at 143.8 103.1 270)
+    (at 147.8 109.1 270)
     (fp_text reference VAL (at 0 0 270) (layer B.SilkS) hide
       (effects (font (size 0.2 0.2) (thickness 0.05)) (justify mirror))
@@
   )
   (module kicad-libraries:WEEE_7mm (layer Rückseite)
-    (at 149.7 99.5 270)
+    (at 147.8 97.6 270)
     (fp_text reference VAL (at 0 0 270) (layer B.SilkS) hide
       (effects (font (size 0.2 0.2) (thickness 0.05)) (justify mirror))
@@
   )
   (module kicad-libraries:Logo_CoMCU (layer Rückseite)
-    (at 150.6 105.6 270)
+    (at 147.8 103.1 270)
     (fp_text reference G*** (at 0 0 270) (layer B.SilkS) hide
       (effects (font (thickness 0.3)) (justify mirror))

Commit message: fix status text
Other:
- board text added: "Status"
- board text removed: "status"
Changed lines of the file:
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@@
     )
   )
-  (gr_text status (at 147.9 91.6) (layer F.SilkS)
+  (gr_text Status (at 147.8 91.6) (layer F.SilkS)
     (effects (font (size 0.7 0.7) (thickness 0.15)))
   )

Commit message: specify processor
Parts:
- U1: value XMC1XXX24 -> XMC11XX24
Changed lines of the file:
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@@
       (effects (font (size 0.3 0.3) (thickness 0.075)))
     )
-    (fp_text value XMC1XXX24 (at 0 0.8 225) (layer F.Fab)
+    (fp_text value XMC11XX24 (at 0 0.8 225) (layer F.Fab)
       (effects (font (size 0.3 0.3) (thickness 0.075)))
     )
